Commit message: add blender files and collada meshes

File: urdf/urdf_test.xacro (robot description, xacro)
@@ -30,6 +30,6 @@
       <origin xyz="0 0 0" rpy="0 0 0"/>
       <geometry>
-        <box size=".4 .2 .15"/>
-        <!--mesh filename = "package://bme_gazebo_sensors/meshes/mogi_bot.dae"/-->
+        <box size=".4 .2 .15"/-->
+        <!--mesh filename = "package://urdf_examples/meshes/base_link.dae"/-->
       </geometry>
       <material name="orange"/>
@@ -65,5 +65,5 @@
       <geometry>
         <cylinder radius="0.05" length=".02"/>
-        <!--mesh filename = "package://bme_gazebo_sensors/meshes/wheel.dae"/-->
+        <!--mesh filename = "package://urdf_examples/meshes/wheel.dae"/-->
       </geometry>
       <material name="green"/>
@@ -98,5 +98,5 @@
       <geometry>
         <cylinder radius="0.05" length=".02"/>
-        <!--mesh filename = "package://bme_gazebo_sensors/meshes/wheel.dae"/-->
+        <!--mesh filename = "package://urdf_examples/meshes/wheel.dae"/-->
       </geometry>
       <material name="green"/>
@@ -131,5 +131,5 @@
       <geometry>
         <cylinder radius="0.05" length=".02"/>
-        <!--mesh filename = "package://bme_gazebo_sensors/meshes/wheel.dae"/-->
+        <!--mesh filename = "package://urdf_examples/meshes/wheel.dae"/-->
       </geometry>
       <material name="green"/>
@@ -164,5 +164,5 @@
       <geometry>
         <cylinder radius="0.05" length=".02"/>
-        <!--mesh filename = "package://bme_gazebo_sensors/meshes/wheel.dae"/-->
+        <!--mesh filename = "package://urdf_examples/meshes/wheel.dae"/-->
       </geometry>
       <material name="green"/>

File: urdf/wheel.xacro (robot description, xacro)
@@ -12,5 +12,5 @@
 				<geometry>
                     <cylinder length="${wheel_length}" radius="${wheel_radius}" />
-					<!--mesh filename="package://husky_description/meshes/wheel.dae" /-->
+                    <!--mesh filename = "package://urdf_examples/meshes/wheel.dae"/-->
 				</geometry>
                 <material name="green"/>

File: urdf/xacro_test.xacro (robot description, xacro)
@@ -46,5 +46,5 @@
       <geometry>
         <box size="${base_x_size} ${base_y_size} ${base_z_size}"/>
-        <!--mesh filename = "package://bme_gazebo_sensors/meshes/mogi_bot.dae"/-->
+        <!--mesh filename = "package://urdf_examples/meshes/base_link.dae"/-->
       </geometry>
       <material name="orange"/>

Commit message: fix a typo

File: urdf/urdf_test.xacro (robot description, xacro)
@@ -30,5 +30,5 @@
       <origin xyz="0 0 0" rpy="0 0 0"/>
       <geometry>
-        <box size=".4 .2 .15"/-->
+        <box size=".4 .2 .15"/>
         <!--mesh filename = "package://urdf_examples/meshes/base_link.dae"/-->
       </geometry>
