Commit message: use meshes instead of basic shapes in xacro

File: urdf/wheel.xacro (robot description, xacro)
@@ -11,6 +11,6 @@
 				<origin xyz="0 0 0" rpy="0 ${M_PI/2} ${M_PI/2}" />
 				<geometry>
-                    <cylinder length="${wheel_length}" radius="${wheel_radius}" />
-                    <!--mesh filename = "package://urdf_examples/meshes/wheel.dae"/-->
+                    <!--cylinder length="${wheel_length}" radius="${wheel_radius}" /-->
+                    <mesh filename = "package://urdf_examples/meshes/wheel.dae"/>
 				</geometry>
                 <material name="green"/>

File: urdf/xacro_test.xacro (robot description, xacro)
@@ -45,6 +45,6 @@
       <origin xyz="0 0 0" rpy="0 0 0"/>
       <geometry>
-        <box size="${base_x_size} ${base_y_size} ${base_z_size}"/>
-        <!--mesh filename = "package://urdf_examples/meshes/base_link.dae"/-->
+        <!--box size="${base_x_size} ${base_y_size} ${base_z_size}"/-->
+        <mesh filename = "package://urdf_examples/meshes/base_link.dae"/>
       </geometry>
       <material name="orange"/>
